File: Projet_Robot_Autonome/ProjetX.kicad_pcb (KiCad board)
At the start: 4 copper layers, 57 x 54 mm, 99 parts, among them IC1 MP1475DJ-LF-P, J1 Conn_ST_STDC14, J11 Conn_01x05, J2 Screw_Terminal_01x02, J3 Conn_01x06, J4 BORDER, J5 Conn_01x06, J6 Conn_01x05, J7 BORDER, J8 BORDER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

Commit message: show errors
Parts:
- moved C1 70.1 mm to (219.9, 139.1)
- moved C10 70.1 mm to (222.1, 132.3)
- moved C11 70.1 mm to (222.1, 131.2)
- moved C22 70.1 mm to (221.0, 137.2)
- moved C3 70.1 mm to (222.2, 126.2)
- moved C5 70.1 mm to (213.3, 124.8)
- moved C6 70.1 mm to (211.3, 134.6)
- moved C7 70.1 mm to (222.0, 128.0)
- moved C8 70.1 mm to (222.0, 130.2)
- moved C9 70.1 mm to (222.0, 129.2)
- moved U1 70.1 mm to (215.9, 130.3)
- moved Y1 70.1 mm to (217.5, 138.6)
- moved C2 70.1 mm to (215.2, 137.9)
- moved R1 70.1 mm to (219.9, 137.2)
- moved C25 34.9 mm to (206.5, 91.1)
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